File: KiCad/Sigini2_main_board/Sigini2_main_board.sch (KiCad schematic (older format))
At the start: 5 parts

Commit message: end build of scheme
Parts:
- removed C?: C, symbol Device:C
- removed SW?: SW_Push_Dual, symbol Switch:SW_Push_Dual
- added C2, C3, C5, C6, C7: 0.1uF, symbol Device:CP
- added C4: 0.47uF, symbol Device:C
- added C8: 33uF, symbol Device:CP
- added J1, J4: Conn_01x03_Male, symbol Connector:Conn_01x03_Male
- added J2: DB9_Male_MountingHoles, symbol Connector:DB9_Male_MountingHoles
- added J3: Conn_01x02_Male, symbol Connector:Conn_01x02_Male
- added R1, R2, R3, R4, R5: 10k, symbol Device:R
- added SW1: SW_Push_Dual, symbol Switch:SW_Push_Dual
- added U3: LM1117-3.3, symbol Regulator_Linear:LM1117-3.3
- C1: renamed from C?; value CP -> 0.1uF
- gave numbers to parts that had none: 2
Connections:
- net labels added: +5V, ESP_RX, ESP_TX
- wire segments 2 -> 84
- no-connect marks 0 -> 19
